Commit message: fix movement issue

File: install/lab_1_package/share/lab_1_package/urdf/robot.urdf (robot description, URDF)
Before this commit: robot my_robot, 7 links, 6 joints
Links:
- removed link depth_camera_link
- removed link front_left_wheel
- removed link front_right_wheel
- removed link rear_left_wheel
- removed link rear_right_wheel
- added link front_left_wheel_link, mass 2.0; collision cylinder length=0.1 radius=0.15; visual cylinder length=0.1 radius=0.15
- added link front_right_wheel_link, mass 2.0; collision cylinder length=0.1 radius=0.15; visual cylinder length=0.1 radius=0.15
- added link rear_left_wheel_link, mass 2.0; collision cylinder length=0.1 radius=0.15; visual cylinder length=0.1 radius=0.15
- added link rear_right_wheel_link, mass 2.0; collision cylinder length=0.1 radius=0.15; visual cylinder length=0.1 radius=0.15
Joints:
- removed joint camera_joint
- removed joint depth_camera_joint
- removed joint front_left_wheel_joint
- removed joint front_right_wheel_joint
- removed joint rear_left_wheel_joint
- removed joint rear_right_wheel_joint
- added joint base_to_camera: type fixed, parent base_link, child camera_link, origin xyz=0.4 0 0.45 rpy=0 0 0
- added joint base_to_front_left_wheel: type continuous, parent base_link, child front_left_wheel_link, origin xyz=0.3 0.35 0.15 rpy=1.57075 0 0, axis 0 0 1
- added joint base_to_front_right_wheel: type continuous, parent base_link, child front_right_wheel_link, origin xyz=0.3 -0.35 0.15 rpy=1.57075 0 0, axis 0 0 1
- added joint base_to_rear_left_wheel: type continuous, parent base_link, child rear_left_wheel_link, origin xyz=-0.3 0.35 0.15 rpy=1.57075 0 0, axis 0 0 1
- added joint base_to_rear_right_wheel: type continuous, parent base_link, child rear_right_wheel_link, origin xyz=-0.3 -0.35 0.15 rpy=1.57075 0 0, axis 0 0 1

Commit message: udpate

File: install/lab_1_package/share/lab_1_package/urdf/robot.urdf (robot description, URDF)
Before this commit: robot my_robot, 6 links, 5 joints
Links:
- removed link front_left_wheel_link
- removed link front_right_wheel_link
- removed link rear_left_wheel_link
- removed link rear_right_wheel_link
- added link depth_camera_link, mass 0.1; visual box size=0.05 0.05 0.05
- added link front_left_wheel, mass 2.0; collision cylinder length=0.1 radius=0.15; visual cylinder length=0.1 radius=0.15
- added link front_right_wheel, mass 2.0; collision cylinder length=0.1 radius=0.15; visual cylinder length=0.1 radius=0.15
- added link rear_left_wheel, mass 2.0; collision cylinder length=0.1 radius=0.15; visual cylinder length=0.1 radius=0.15
- added link rear_right_wheel, mass 2.0; collision cylinder length=0.1 radius=0.15; visual cylinder length=0.1 radius=0.15
Joints:
- removed joint base_to_camera
- removed joint base_to_front_left_wheel
- removed joint base_to_front_right_wheel
- removed joint base_to_rear_left_wheel
- removed joint base_to_rear_right_wheel
- added joint camera_joint: type fixed, parent base_link, child camera_link, origin xyz=0.4 0 0.45 rpy=0 0 0
- added joint depth_camera_joint: type fixed, parent base_link, child depth_camera_link, origin xyz=0.4 0 0.45 rpy=0 0 0
- added joint front_left_wheel_joint: type continuous, parent base_link, child front_left_wheel, origin xyz=0.3 0.35 0.15 rpy=1.57075 0 0, axis 0 0 1
- added joint front_right_wheel_joint: type continuous, parent base_link, child front_right_wheel, origin xyz=0.3 -0.35 0.15 rpy=1.57075 0 0, axis 0 0 1
- added joint rear_left_wheel_joint: type continuous, parent base_link, child rear_left_wheel, origin xyz=-0.3 0.35 0.15 rpy=1.57075 0 0, axis 0 0 1
- added joint rear_right_wheel_joint: type continuous, parent base_link, child rear_right_wheel, origin xyz=-0.3 -0.35 0.15 rpy=1.57075 0 0, axis 0 0 1
